Commit message: Fix simulation blockers: missing macro call, TF chain, missing world file, gzclient crash
- ackermann.xacro: invoke the limo_ackermann macro (was defined but never
  called, so base_link and the whole chassis never made it into the URDF)
- ackermann.xacro: uncomment base_footprint link + base_joint so the TF
  tree connects to the odom->base_footprint transform published by the
  ackermann_controller plugin (previously two disconnected TF trees)
- ackermann_with_sensor.xacro: disable the depth camera sensor, which
  crashes gzserver with a rendering::Scene assertion on spawn regardless
  of display session or renderer
- worlds/empty_world.model: add the world file referenced by
  ackermann_gazebo.launch.py that was missing from the repo entirely
  (gzserver would hang trying to open a nonexistent file), plus a few
  box obstacles for LiDAR to actually see something
- .gitignore: un-ignore *.model files under limo_car/worlds/ (a generic
  kernel-module *.mod* pattern was silently eating the world file above)
- ackermann_gazebo.launch.py: run gzserver/gzclient separately instead of
  through gazebo.launch.py, since the latter hardcodes
  --gui-client-plugin=libgazebo_ros_eol_gui.so which crashes gzclient
  with a Camera assertion on spawn; delay spawn_entity so gzclient has
  time to initialize its own camera first
- rviz/gazebo.rviz: rewrite from scratch (previous file failed to load
  with "Invalid argument" and had no RobotModel/TF display at all)

Co-Authored-By: Claude Sonnet 5 <noreply@anthropic.com>

File: limo_car/gazebo/ackermann.xacro (robot description, xacro)
@@ -204,10 +204,10 @@
     Darstellungspostion in Simulation-Umgebung -->
     <xacro:macro name="limo_ackermann">
-        <!-- <link name="base_footprint"/>
+        <link name="base_footprint"/>
         <joint name="base_joint" type="fixed">
             <parent link="base_footprint"/>
             <child link="base_link"/>
             <origin xyz="0.0 0.0 0.15" rpy="0 0 0"/>
-        </joint> -->
+        </joint>
         <!-- herstellt base_link -->
         <link name="base_link">

File: limo_car/gazebo/ackermann_with_sensor.xacro (robot description, xacro)
@@ -9,4 +9,5 @@
     <xacro:include filename="$(find limo_car)/gazebo/ackermann.xacro" />
     <xacro:include filename="$(find limo_car)/gazebo/sensor.xacro" />
+    <xacro:limo_ackermann/>
     <!-- ************************* Laser ****************************** -->
     <xacro:gazebo_laser frame_prefix="laser" />
@@ -17,4 +18,8 @@
     </joint>
     <!-- ************************* Depth-camera *********************** -->
+    <!-- Disabled: this camera sensor crashes gzserver (rendering::Scene
+         assertion) as soon as the model is spawned, independent of the
+         display session (X11/Wayland) or the gzclient EOL-plugin fix. -->
+    <!--
     <xacro:gazebo_depth_camera frame_prefix="depth_camera" />
     <joint name="depth_camera_joint" type="fixed">
@@ -23,4 +28,5 @@
         <child link="depth_camera_link"/>
     </joint>
+    -->
     <!-- ************************* IMU ******************************** -->
     <xacro:gazebo_imu frame_prefix="imu" />

Commit message: Lightweight single-mesh body/wheel + fix depth camera crash via xvfb
- Replace limo_base.dae (1619 sub-meshes, 755K faces) and limo_wheel.dae
  (3 sub-meshes, 140K faces) with single welded+decimated STL meshes
  (~98K and ~12K faces respectively). The fragmentation into hundreds of
  separate draw calls, not raw polygon count, was the source of the
  reported Gazebo/RViz stuttering.
- Body and wheels now use flat colors (Gazebo/Grey, Gazebo/Black) via
  <gazebo reference="link_name"><material>...</material></gazebo>
  instead of per-visual URDF <material><color> tags, which Gazebo
  Classic silently ignores for mesh geometries.
- ackermann_gazebo.launch.py: run gzserver under xvfb-run (isolated
  virtual X display). The depth camera sensor was crashing gzserver
  with a rendering::Scene assertion on spawn regardless of the real
  session's display server (X11/Wayland) or GPU driver config; giving
  it its own clean virtual display avoids whatever conflict that was.
  Depth camera re-enabled now that this works.

Co-Authored-By: Claude Sonnet 5 <noreply@anthropic.com>

File: limo_car/gazebo/ackermann.xacro (robot description, xacro)
@@ -96,6 +96,9 @@
                 <origin xyz="0 0 0" rpy="0 0 0" />
                 <geometry>
-                    <mesh filename="$(find limo_car)/meshes/limo_wheel.dae" scale="1.2 1.2 1.2"/>
-                </geometry>
+                    <mesh filename="$(find limo_car)/meshes/limo_wheel_lean.stl" scale="1.2 1.2 1.2"/>
+                </geometry>
+                <material name="wheel_black">
+                    <color rgba="0.1 0.1 0.1 1"/>
+                </material>
             </visual>
             <collision>
@@ -107,4 +110,7 @@
             <xacro:cylinder_inertial_matrix  m="${wheel_mass}" r="${wheel_radius}"  h="${wheel_length}" />
         </link>
+        <gazebo reference="${wheel_prefix}_wheel_link">
+            <material>Gazebo/Black</material>
+        </gazebo>
         <joint name="${wheel_prefix}_wheel_joint" type="continuous">
             <parent link="${wheel_prefix}_steer_link"/>
@@ -168,6 +174,9 @@
                 <origin xyz="0 0 0" rpy="0 0 0" />
                 <geometry>
-                    <mesh filename="$(find limo_car)/meshes/limo_wheel.dae" scale="1.2 1.2 1.2" />
-                </geometry>
+                    <mesh filename="$(find limo_car)/meshes/limo_wheel_lean.stl" scale="1.2 1.2 1.2" />
+                </geometry>
+                <material name="wheel_black">
+                    <color rgba="0.1 0.1 0.1 1"/>
+                </material>
             </visual>
             <collision>
@@ -179,4 +188,7 @@
             <xacro:cylinder_inertial_matrix  m="${wheel_mass}" r="${wheel_radius}"  h="${wheel_length}" />
         </link>
+        <gazebo reference="${wheel_prefix}_wheel_link">
+            <material>Gazebo/Black</material>
+        </gazebo>
         <joint name="${wheel_prefix}_wheel_joint" type="continuous">
             <parent link="${wheel_prefix}_steer_link"/>
@@ -211,11 +223,17 @@
         </joint>
         <!-- herstellt base_link -->
+        <!-- Leichtgewichtige Version: limo_base.dae bestand aus 1619
+             einzelnen Sub-Meshes (755K Faces), was zu massivem Ruckeln
+             führte (viele Draw-Calls). Hier zu einem Mesh verschmolzen und
+             dezimiert (~98K Faces), einfarbig. -->
         <link name="base_link">
             <visual>
                 <origin xyz="0 0 -0.15" rpy="0 0 ${M_PI/2}" />
                 <geometry>
-                    <!-- Modell von Hersteller, aber es ist kleiner als realen Produkt, da die Skale vergrößert wird -->
-                    <mesh filename="$(find limo_car)/meshes/limo_base.dae" scale="1.2 1.2 1.2" />
-                </geometry>
+                    <mesh filename="$(find limo_car)/meshes/limo_base_lean.stl" scale="1.2 1.2 1.2" />
+                </geometry>
+                <material name="body_white">
+                    <color rgba="0.9 0.9 0.9 1"/>
+                </material>
             </visual>
             <!-- Modell für physikalische Kollision zu modellieren. -->
@@ -229,7 +247,5 @@
         </link>
         <gazebo reference="base_link">
-            <material>
-                <color rgba="0 0 0 0.5"/>
-            </material>
+            <material>Gazebo/Grey</material>
         </gazebo>
         <!-- hinten Räder -->
@@ -238,6 +254,9 @@
                 <origin xyz="0 0 0" rpy="0 0 0" />
                 <geometry>
-                    <mesh filename="$(find limo_car)/meshes/limo_wheel.dae" scale="1.2 1.2 1.2"/>
-                </geometry>
+                    <mesh filename="$(find limo_car)/meshes/limo_wheel_lean.stl" scale="1.2 1.2 1.2"/>
+                </geometry>
+                <material name="wheel_black">
+                    <color rgba="0.1 0.1 0.1 1"/>
+                </material>
             </visual>
             <collision>
@@ -249,4 +268,7 @@
             <xacro:cylinder_inertial_matrix  m="${wheel_mass}" r="${wheel_radius}" h="${wheel_length}"/>
         </link>
+        <gazebo reference="rear_left_wheel_link">
+            <material>Gazebo/Black</material>
+        </gazebo>
         <joint name="rear_left_wheel_joint" type="continuous">
             <parent link="base_link"/>
@@ -269,6 +291,9 @@
                 <origin xyz="0 0 0" rpy="0 0 0" />
                 <geometry>
-                    <mesh filename="$(find limo_car)/meshes/limo_wheel.dae" scale="1.2 1.2 1.2"/>
-                </geometry>
+                    <mesh filename="$(find limo_car)/meshes/limo_wheel_lean.stl" scale="1.2 1.2 1.2"/>
+                </geometry>
+                <material name="wheel_black">
+                    <color rgba="0.1 0.1 0.1 1"/>
+                </material>
             </visual>
             <collision>
@@ -280,4 +305,7 @@
             <xacro:cylinder_inertial_matrix  m="${wheel_mass}" r="${wheel_radius}" h="${wheel_length}"/>
         </link>
+        <gazebo reference="rear_right_wheel_link">
+            <material>Gazebo/Black</material>
+        </gazebo>
         <joint name="rear_right_wheel_joint" type="continuous">
             <parent link="base_link"/>

File: limo_car/gazebo/ackermann_with_sensor.xacro (robot description, xacro)
@@ -18,8 +18,4 @@
     </joint>
     <!-- ************************* Depth-camera *********************** -->
-    <!-- Disabled: this camera sensor crashes gzserver (rendering::Scene
-         assertion) as soon as the model is spawned, independent of the
-         display session (X11/Wayland) or the gzclient EOL-plugin fix. -->
-    <!--
     <xacro:gazebo_depth_camera frame_prefix="depth_camera" />
     <joint name="depth_camera_joint" type="fixed">
@@ -28,5 +24,4 @@
         <child link="depth_camera_link"/>
     </joint>
-    -->
     <!-- ************************* IMU ******************************** -->
     <xacro:gazebo_imu frame_prefix="imu" />

File: limo_car/gazebo/sensor.xacro (robot description, xacro)
@@ -118,5 +118,5 @@
                 <pose>0.0 0.0 0.0 0.0 0.0 0.0</pose>
                 <always_on>true</always_on>
-                <visualize>true</visualize>
+                <visualize>false</visualize>
                 <update_rate>10.0</update_rate>
                 <camera name="head">

Commit message: Speed up steering response - raise steer joint velocity limit
User reported steering felt too slow to respond in sim. Root cause:
front_left/right_steer_joint had <limit velocity="0.5"/> (rad/s) in
ackermann.xacro. That's a hard physics cap Gazebo enforces regardless
of the ackermann_drive plugin's steering PID gain (already stiff,
P=10000) - going from center to full lock (max_steer=0.5236 rad, 30
degrees) took over a second no matter how hard the PID pushed, which
reads as sluggish/laggy steering even though the commanded angle
itself is set instantly (dashboard side was already fixed to be
instant-response in an earlier change).

Raise velocity to 3.0 rad/s (~0.17s to full lock) on both steering
hinge joints, and bump effort 5->10 so the joint can actually reach
that speed against its damping/friction (1.0/2.0) - the old effort=5
was right at the edge of what's needed to sustain 0.5 rad/s already,
not enough headroom for 3.0.

ackermann_with_sensor.xacro includes this file directly, so the fix
applies to the sensor-equipped robot too. Verified all urdf/gazebo
xacro files still process cleanly after the edit.

Co-Authored-By: Claude Sonnet 5 <noreply@anthropic.com>

File: limo_car/gazebo/ackermann.xacro (robot description, xacro)
@@ -79,5 +79,10 @@
             <axis xyz="0 0 1" />
             <!-- Paramenten von Herstellern -->
-            <limit lower="-0.523598767" upper="0.523598767" effort="5" velocity="0.5" />
+            <!-- velocity war 0.5 rad/s - bei max_steer=0.5236 rad dauert ein
+                 Volleinschlag damit >1s, spuerbar traege trotz hohem PID-Gain
+                 im ackermann_drive plugin (P=10000). Auf 3.0 rad/s angehoben
+                 (~0.17s bis Anschlag), effort mit angehoben damit das Limit
+                 gegen damping/friction auch erreichbar ist. -->
+            <limit lower="-0.523598767" upper="0.523598767" effort="10" velocity="3.0" />
             <dynamics damping="1.0" friction="2.0"/>
         </joint>
@@ -157,5 +162,5 @@
             <xacro:insert_block name="joint_pose"/>
             <axis xyz="0 0 -1"/>
-            <limit lower="-0.523598767" upper="0.523598767" effort="5" velocity="0.5" />
+            <limit lower="-0.523598767" upper="0.523598767" effort="10" velocity="3.0" />
             <dynamics damping="1.0" friction="2.0"/>
         </joint>
